File: schematic/clock/clock.kicad_sch (KiCad schematic)
At the start: 20 parts, among them J1 Conn_01x02_Socket, J2 Conn_01x04_Socket, U1 NE555P, U2 ATF16V8B

Commit message: Update schematic
Parts:
- added U2:04: ATF16V8, symbol 74xx:74LS08
- added U2:14: ATF16V8, symbol 74xx:74LS04
- added U2:16, U2:17, U2:x2, U2:x4: ~, symbol 74xx:74LS32
- added U2:19: ~, symbol 74xGxx:74AUC2G79
- added U2:2, U2:9, U2:x0, U2:x5, U3: ~, symbol 74xx:74LS08
Connections:
- net HLT: now also U2:9.9
- net CLKOUT renamed CLKLED
- net CLKLED: now also U2:9.12
- new net: U2:17., U3.
- new net: U2:x4., U2:x5.
- new net: U2:9., U2:x2.
- new net: U2:x2., U2:x5.
- new net: U2:2., U2:x2.
- new net: U2:04., U2:16.
- new net: U2:17., U2:x0.
- new net (DEB_{PUSH}): U2:17.17, U2:19. (D), U2:x0., U2:x4.
- new net (FF_{HOLD}): U2:19.19 (Q), U2:x0., U2:x4.
- new net CLK: U2:19.1 (C)
- new net CLKI: U2:2.2
- new net DEB_{MAUTO}: U2:04., U2:14., U2:16.16, U2:2.
- new net DEB_{MMAN}: U2:14.14, U2:x5., U3.
- new net PUSH: U3.3
- new net ~{MAUTO}: U2:16.5
- new net ~{MMAN}: U2:04.4
Other:
- note added: "13"
- note added: "15"
- note added: "Logic programmed into U2 [ATF16V8B SPLD]"
- moved on the sheet: BUT1, C1, C2, J1, J2, LED1, LEDI1, LEDI2, POT1, R1, R2, RL1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

Commit message: Add schematic title/date
Connections:
- net at U2:17.: now also U2:x0.; no longer U3.
- net at U2:x2.: now also U2:2.; no longer U2:x5.
- new net: U2:17., U3.
- new net: U2:x4., U2:x5.
- new net: U2:x2., U2:x5.
Other:
- company: (none) -> Silicon Chronicles
Changed lines of the file:
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@@
 	(title_block
 		(title "Debug Clock Module")
+		(date "2024-05-06")
+		(company "Silicon Chronicles")
 	)
 	(junction
